File: lever-arena.sch (EAGLE design)
At the start: 6 parts, among them Q1 FQP30N06L, Q2 FQP30N06L

Commit message: added all components
Parts:
- removed Q1, Q2: FQP30N06L, spencer:FQP30N06L
- removed U$1: MCP3208, spencer:MCP3208
- added ADC0: MCP3208, spencer:MCP3208
- added D1, D2: 1N4148, SparkFun-DiscreteSemi:DIODE1N4148
- added HL0, HL1, HR0, HR1, VL0, VL1, VR0, VR1: (no value), pinhead:PINHD-1X6
- added J1: POWER_JACKPTH, SparkFun-Connectors:POWER_JACKPTH
- added MOSFET0, MOSFET1: MOSFET-NCHANNELFQP30N06L, SparkFun-DiscreteSemi:MOSFET-NCHANNELFQP30N06L
- added PUMP0, PUMP1: (no value), pinhead:PINHD-1X2
- added R1, R2: 10k, SparkFun-Resistors:10KOHM-1/4W-1%(PTH)HORIZ
- renumbered U$2 to ADC1
Connections:
- removed net N$2: U$1.AGND
- new net 12V: D1.C, D2.A, D2.C, J1.PWR, JP1.VIN, MOSFET1.D, PUMP0.1, PUMP1.1, PUMP1.2
- new net 3V3: ADC0.VREF, ADC1.VREF, PCB1.3V3@1, PCB1.3V3@17
- new net A1: PCB1.GPIO5
- new net A2: PCB1.GPIO6
- new net A3: PCB1.GPIO13
- new net A4: PCB1.GPIO19
- new net A5: PCB1.GPIO26
- new net A6: PCB1.GPIO16
- new net A7: PCB1.GPIO20
- new net A8: PCB1.GPIO21
- new net HL0: HL0.3
- new net HL1: HL1.3
- new net HR0: HR0.3
- new net HR1: HR1.3
- new net N$1: ADC1.CH1, VL1.4
- new net N$11: PCB1.GPIO18
- new net N$12: PCB1.GND@14
- new net N$13: PCB1.GPIO23
- new net N$14: PCB1.GPIO24
- new net N$15: PCB1.GND@20
- new net N$16: PCB1.GPIO25
- new net N$17: PCB1.ID_SC*
- new net N$18: PCB1.GND@30
- new net N$19: PCB1.GPIO12
- new net N$20: PCB1.GND@34
- new net N$21: ADC1.CH3, HR1.4
- new net N$22: ADC1.CH7, HL0.4
- new net N$23: ADC1.CH6, VL0.4
- new net N$24: ADC0.CH5
- new net N$25: ADC0.CH6
- new net N$26: ADC0.CH7
- new net N$27: ADC1.CH5, VR0.4
- new net N$28: ADC1.CH4, HR0.4
- new net N$3: ADC1.CH2, VR1.4
- new net N$30: PCB1.ID_SD*
- new net N$32: PCB1.GPIO22
- new net N$33: PCB1.GPIO27
- new net N$34: PCB1.GPIO17
- new net N$36: PCB1.GPIO4
- new net N$37: PCB1.GPIO3
- new net N$38: PCB1.GPIO2
- new net N$4: D1.A, MOSFET0.D, PUMP0.2
- new net N$48: ADC1.CH0, HL1.4
- new net N$5: ADC0.CH0
- new net N$6: ADC0.CH1
- new net N$7: ADC0.CH2
- new net N$8: JP1.EN
- new net PUMP1: MOSFET0.G, PCB1.GPIO14, R2.1
- new net PUMP2: MOSFET1.G, PCB1.GPIO15, R1.1
- new net VL0: VL0.3
- new net VL1: VL1.3
- new net VR0: VR0.3
- new net VR1: VR1.3
- net 5V: now also ADC0.VDD, ADC1.VDD, HL0.2, HL1.2, HR0.2, HR1.2, VL0.2, VL1.2, VR0.2, VR1.2
- net CE0: now also ADC0.CS; no longer U$1.CS
- net GND: now also ADC0.AGND, ADC0.DGND, ADC1.AGND, ADC1.DGND, HL0.1, HL1.1, HR0.1, HR1.1, J1.GND, MOSFET0.S, MOSFET1.S, PCB1.GND@25, PCB1.GND@39, PCB1.GND@9, R1.2, R2.2, VL0.1, VL1.1, VR0.1, VR1.1
- net MISO: now also ADC0.DOUT; no longer U$1.DOUT
- net MOSI: now also ADC0.DIN; no longer U$1.DIN
- net N$10: now also ADC0.CH4; no longer ADC1.DGND
- net N$9: now also ADC0.CH3; no longer U$1.DGND
- net SCLK: now also ADC0.CLK; no longer U$1.CLK

Commit message: Updated
Parts:
- added JP2, JP3, JP4: (no value), pinhead:PINHD-1X8
- J1: value POWER_JACKPTH -> POWER_JACKPTH_BREAD; device SparkFun-Connectors:POWER_JACKPTH -> SparkFun-Connectors:POWER_JACKPTH_BREAD
Connections:
- net A8 renamed N$3
- removed net A1: PCB1.GPIO5
- removed net A2: PCB1.GPIO6
- removed net A3: PCB1.GPIO13
- removed net A4: PCB1.GPIO19
- removed net A5: PCB1.GPIO26
- removed net A6: PCB1.GPIO16
- removed net A7: PCB1.GPIO20
- removed net N$1: ADC1.CH1, VL1.4
- removed net N$11: PCB1.GPIO18
- removed net N$12: PCB1.GND@14
- removed net N$13: PCB1.GPIO23
- removed net N$14: PCB1.GPIO24
- removed net N$15: PCB1.GND@20
- removed net N$16: PCB1.GPIO25
- removed net N$17: PCB1.ID_SC*
- removed net N$18: PCB1.GND@30
- removed net N$19: PCB1.GPIO12
- removed net N$20: PCB1.GND@34
- removed net N$21: ADC1.CH3, HR1.4
- removed net N$3 (its old number): ADC1.CH2, VR1.4
- removed net N$30: PCB1.ID_SD*
- removed net N$34: PCB1.GPIO17
- removed net N$36: PCB1.GPIO4
- removed net N$37: PCB1.GPIO3
- removed net N$38: PCB1.GPIO2
- removed net N$48: ADC1.CH0, HL1.4
- new net N$29: ADC1.CH0, HR1.4
- new net N$31: ADC1.CH1, VR1.4
- net 3V3: no longer PCB1.3V3@1
- net GND: no longer PCB1.GND@39, PCB1.GND@6
- net HL0: now also PCB1.GPIO5
- net HL1: now also PCB1.GPIO16
- net HR0: now also PCB1.GPIO13
- net HR1: now also PCB1.GPIO26
- net N$32: now also ADC1.CH2, VL1.4; no longer PCB1.GPIO22
- net N$33: now also ADC1.CH3, HL1.4; no longer PCB1.GPIO27
- net PUMP1: now also PCB1.GPIO17; no longer PCB1.GPIO14
- net PUMP2: now also PCB1.GPIO27; no longer PCB1.GPIO15
- net VL0: now also PCB1.GPIO6
- net VL1: now also PCB1.GPIO19
- net VR0: now also PCB1.GPIO12
- net VR1: now also PCB1.GPIO20
Other:
- moved on the sheet: HL1, HR1, VL1, VR1

Commit message: All connectors added
Parts:
- removed JP2, JP3, JP4: (no value), pinhead:PINHD-1X8
- added 3V3, AIN, GND: (no value), pinhead:PINHD-1X8
Connections:
- removed net N$10: ADC0.CH4
- removed net N$24: ADC0.CH5
- removed net N$25: ADC0.CH6
- removed net N$26: ADC0.CH7
- removed net N$5: ADC0.CH0
- removed net N$6: ADC0.CH1
- removed net N$7: ADC0.CH2
- removed net N$9: ADC0.CH3
- new net N$1: ADC0.CH0, AIN.1
- new net N$11: ADC0.CH1, AIN.2
- new net N$12: ADC0.CH2, AIN.3
- new net N$13: ADC0.CH3, AIN.4
- new net N$14: ADC0.CH4, AIN.5
- new net N$15: ADC0.CH5, AIN.6
- new net N$16: ADC0.CH6, AIN.7
- new net N$17: ADC0.CH7, AIN.8
- net 3V3: now also 3V3.1, 3V3.2, 3V3.3, 3V3.4, 3V3.5, 3V3.6, 3V3.7, 3V3.8, PCB1.3V3@1
- net GND: now also GND.1, GND.2, GND.3, GND.4, GND.5, GND.6, GND.7, GND.8
Changed lines of the file:
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@@
 <part name="VR0" library="pinhead" deviceset="PINHD-1X6" device=""/>
 <part name="HR0" library="pinhead" deviceset="PINHD-1X6" device=""/>
-<part name="JP2" library="pinhead" deviceset="PINHD-1X8" device=""/>
-<part name="JP3" library="pinhead" deviceset="PINHD-1X8" device=""/>
-<part name="JP4" library="pinhead" deviceset="PINHD-1X8" device=""/>
+<part name="GND" library="pinhead" deviceset="PINHD-1X8" device=""/>
+<part name="AIN" library="pinhead" deviceset="PINHD-1X8" device=""/>
+<part name="3V3" library="pinhead" deviceset="PINHD-1X8" device=""/>
 </parts>
 <sheets>
@@
 <instance part="VR0" gate="A" x="17.78" y="-127" rot="MR180"/>
 <instance part="HR0" gate="A" x="17.78" y="-149.86" rot="MR180"/>
-<instance part="JP2" gate="A" x="-88.9" y="-83.82" rot="R180"/>
-<instance part="JP3" gate="A" x="-101.6" y="-86.36"/>
-<instance part="JP4" gate="A" x="-71.12" y="-83.82" rot="R180"/>
+<instance part="GND" gate="A" x="-76.2" y="-86.36"/>
+<instance part="AIN" gate="A" x="-71.12" y="-86.36" rot="MR0"/>
+<instance part="3V3" gate="A" x="-93.98" y="-86.36"/>
 </instances>
 <busses>
@@
 <label x="20.32" y="-157.48" size="1.27" layer="95" rot="MR180" xref="yes"/>
 </segment>
+<segment>
+<pinref part="GND" gate="A" pin="1"/>
+<junction x="-78.74" y="-76.2"/>
+<label x="-83.82" y="-76.2" size="1.27" layer="95" rot="R180" xref="yes"/>
+</segment>
+<segment>
+<pinref part="GND" gate="A" pin="2"/>
+<junction x="-78.74" y="-78.74"/>
+<label x="-83.82" y="-78.74" size="1.27" layer="95" rot="R180" xref="yes"/>
+</segment>
+<segment>
+<pinref part="GND" gate="A" pin="3"/>
+<junction x="-78.74" y="-81.28"/>
+<label x="-83.82" y="-81.28" size="1.27" layer="95" rot="R180" xref="yes"/>
+</segment>
+<segment>
+<pinref part="GND" gate="A" pin="5"/>
+<junction x="-78.74" y="-86.36"/>
+<label x="-83.82" y="-86.36" size="1.27" layer="95" rot="R180" xref="yes"/>
+</segment>
+<segment>
+<pinref part="GND" gate="A" pin="4"/>
+<junction x="-78.74" y="-83.82"/>
+<label x="-83.82" y="-83.82" size="1.27" layer="95" rot="R180" xref="yes"/>
+</segment>
+<segment>
+<pinref part="GND" gate="A" pin="6"/>
+<junction x="-78.74" y="-88.9"/>
+<label x="-83.82" y="-88.9" size="1.27" layer="95" rot="R180" xref="yes"/>
+</segment>
+<segment>
+<pinref part="GND" gate="A" pin="7"/>
+<junction x="-78.74" y="-91.44"/>
+<label x="-83.82" y="-91.44" size="1.27" layer="95" rot="R180" xref="yes"/>
+</segment>
+<segment>
+<pinref part="GND" gate="A" pin="8"/>
+<junction x="-78.74" y="-93.98"/>
+<label x="-83.82" y="-93.98" size="1.27" layer="95" rot="R180" xref="yes"/>
+</segment>
 </net>
 <net name="3V3" class="0">
@@
 <junction x="-7.62" y="-12.7"/>
 <label x="-7.62" y="-15.24" size="1.27" layer="95" rot="R270" xref="yes"/>
+</segment>
+<segment>
+<pinref part="3V3" gate="A" pin="1"/>
+<junction x="-96.52" y="-76.2"/>
+<label x="-101.6" y="-76.2" size="1.27" layer="95" rot="R180" xref="yes"/>
+</segment>
+<segment>
+<pinref part="3V3" gate="A" pin="2"/>
+<junction x="-96.52" y="-78.74"/>
+<label x="-101.6" y="-78.74" size="1.27" layer="95" rot="R180" xref="yes"/>
+</segment>
+<segment>
+<pinref part="3V3" gate="A" pin="3"/>
+<junction x="-96.52" y="-81.28"/>
+<label x="-101.6" y="-81.28" size="1.27" layer="95" rot="R180" xref="yes"/>
+</segment>
+<segment>
+<pinref part="3V3" gate="A" pin="4"/>
+<junction x="-96.52" y="-83.82"/>
+<label x="-101.6" y="-83.82" size="1.27" layer="95" rot="R180" xref="yes"/>
+</segment>
+<segment>
+<pinref part="3V3" gate="A" pin="5"/>
+<junction x="-96.52" y="-86.36"/>
+<label x="-101.6" y="-86.36" size="1.27" layer="95" rot="R180" xref="yes"/>
+</segment>
+<segment>
+<pinref part="3V3" gate="A" pin="6"/>
+<junction x="-96.52" y="-88.9"/>
+<label x="-101.6" y="-88.9" size="1.27" layer="95" rot="R180" xref="yes"/>
+</segment>
+<segment>
+<pinref part="3V3" gate="A" pin="7"/>
+<junction x="-96.52" y="-91.44"/>
+<label x="-101.6" y="-91.44" size="1.27" layer="95" rot="R180" xref="yes"/>
+</segment>
+<segment>
+<pinref part="3V3" gate="A" pin="8"/>
+<junction x="-96.52" y="-93.98"/>
+<label x="-101.6" y="-93.98" size="1.27" layer="95" rot="R180" xref="yes"/>
+</segment>
+<segment>
+<pinref part="PCB1" gate="G$1" pin="3V3@1"/>
+<junction x="-48.26" y="-12.7"/>
+<label x="-48.26" y="-15.24" size="1.27" layer="95" rot="R270" xref="yes"/>
 </segment>
 </net>
@@
 </segment>
 </net>
-<net name="N$5" class="0">
-<segment>
-<pinref part="ADC0" gate="MCP3208$1" pin="CH0"/>
-<junction x="-60.96" y="-68.58"/>
-</segment>
-</net>
-<net name="N$6" class="0">
-<segment>
-<pinref part="ADC0" gate="MCP3208$1" pin="CH1"/>
-<junction x="-58.42" y="-68.58"/>
-</segment>
-</net>
-<net name="N$7" class="0">
-<segment>
-<pinref part="ADC0" gate="MCP3208$1" pin="CH2"/>
-<junction x="-55.88" y="-68.58"/>
-</segment>
-</net>
-<net name="N$9" class="0">
-<segment>
-<pinref part="ADC0" gate="MCP3208$1" pin="CH3"/>
-<junction x="-53.34" y="-68.58"/>
-</segment>
-</net>
-<net name="N$10" class="0">
-<segment>
-<pinref part="ADC0" gate="MCP3208$1" pin="CH4"/>
-<junction x="-50.8" y="-68.58"/>
-</segment>
-</net>
-<net name="N$24" class="0">
-<segment>
-<pinref part="ADC0" gate="MCP3208$1" pin="CH5"/>
-<junction x="-48.26" y="-68.58"/>
-</segment>
-</net>
-<net name="N$25" class="0">
-<segment>
-<pinref part="ADC0" gate="MCP3208$1" pin="CH6"/>
-<junction x="-45.72" y="-68.58"/>
-</segment>
-</net>
-<net name="N$26" class="0">
-<segment>
-<pinref part="ADC0" gate="MCP3208$1" pin="CH7"/>
-<junction x="-43.18" y="-68.58"/>
-</segment>
-</net>
 <net name="HR0" class="0">
 <segment>
@@
 </segment>
 </net>
+<net name="N$1" class="0">
+<segment>
+<pinref part="AIN" gate="A" pin="1"/>
+<junction x="-68.58" y="-76.2"/>
+<pinref part="ADC0" gate="MCP3208$1" pin="CH0"/>
+<junction x="-60.96" y="-68.58"/>
+<wire x1="-68.58" y1="-76.2" x2="-60.96" y2="-76.2" width="0.1524" layer="91"/>
+<wire x1="-60.96" y1="-76.2" x2="-60.96" y2="-68.58" width="0.1524" layer="91"/>
+</segment>
+</net>
+<net name="N$11" class="0">
+<segment>
+<pinref part="AIN" gate="A" pin="2"/>
+<junction x="-68.58" y="-78.74"/>
+<pinref part="ADC0" gate="MCP3208$1" pin="CH1"/>
+<junction x="-58.42" y="-68.58"/>
+<wire x1="-68.58" y1="-78.74" x2="-58.42" y2="-78.74" width="0.1524" layer="91"/>
+<wire x1="-58.42" y1="-78.74" x2="-58.42" y2="-68.58" width="0.1524" layer="91"/>
+</segment>
+</net>
+<net name="N$12" class="0">
+<segment>
+<pinref part="AIN" gate="A" pin="3"/>
+<junction x="-68.58" y="-81.28"/>
+<pinref part="ADC0" gate="MCP3208$1" pin="CH2"/>
+<junction x="-55.88" y="-68.58"/>
+<wire x1="-68.58" y1="-81.28" x2="-55.88" y2="-81.28" width="0.1524" layer="91"/>
+<wire x1="-55.88" y1="-81.28" x2="-55.88" y2="-68.58" width="0.1524" layer="91"/>
+</segment>
+</net>
+<net name="N$13" class="0">
+<segment>
+<pinref part="AIN" gate="A" pin="4"/>
+<junction x="-68.58" y="-83.82"/>
+<pinref part="ADC0" gate="MCP3208$1" pin="CH3"/>
+<junction x="-53.34" y="-68.58"/>
+<wire x1="-68.58" y1="-83.82" x2="-53.34" y2="-83.82" width="0.1524" layer="91"/>
+<wire x1="-53.34" y1="-83.82" x2="-53.34" y2="-68.58" width="0.1524" layer="91"/>
+</segment>
+</net>
+<net name="N$14" class="0">
+<segment>
+<pinref part="AIN" gate="A" pin="5"/>
+<junction x="-68.58" y="-86.36"/>
+<pinref part="ADC0" gate="MCP3208$1" pin="CH4"/>
+<junction x="-50.8" y="-68.58"/>
+<wire x1="-68.58" y1="-86.36" x2="-50.8" y2="-86.36" width="0.1524" layer="91"/>
+<wire x1="-50.8" y1="-86.36" x2="-50.8" y2="-68.58" width="0.1524" layer="91"/>
+</segment>
+</net>
+<net name="N$15" class="0">
+<segment>
+<pinref part="AIN" gate="A" pin="6"/>
+<junction x="-68.58" y="-88.9"/>
+<pinref part="ADC0" gate="MCP3208$1" pin="CH5"/>
+<junction x="-48.26" y="-68.58"/>
+<wire x1="-68.58" y1="-88.9" x2="-48.26" y2="-88.9" width="0.1524" layer="91"/>
+<wire x1="-48.26" y1="-88.9" x2="-48.26" y2="-68.58" width="0.1524" layer="91"/>
+</segment>
+</net>
+<net name="N$16" class="0">
+<segment>
+<pinref part="AIN" gate="A" pin="7"/>
+<junction x="-68.58" y="-91.44"/>
+<pinref part="ADC0" gate="MCP3208$1" pin="CH6"/>
+<junction x="-45.72" y="-68.58"/>
+<wire x1="-68.58" y1="-91.44" x2="-45.72" y2="-91.44" width="0.1524" layer="91"/>
+<wire x1="-45.72" y1="-91.44" x2="-45.72" y2="-68.58" width="0.1524" layer="91"/>
+</segment>
+</net>
+<net name="N$17" class="0">
+<segment>
+<pinref part="AIN" gate="A" pin="8"/>
+<junction x="-68.58" y="-93.98"/>
+<pinref part="ADC0" gate="MCP3208$1" pin="CH7"/>
+<junction x="-43.18" y="-68.58"/>
+<wire x1="-68.58" y1="-93.98" x2="-43.18" y2="-93.98" width="0.1524" layer="91"/>
+<wire x1="-43.18" y1="-93.98" x2="-43.18" y2="-68.58" width="0.1524" layer="91"/>
+</segment>
+</net>

Commit message: REVISION 2.2
Parts:
- 3V3: value (none) -> 3v3
- AIN: value (none) -> AIN
- GND: value (none) -> GND
- HL0: value (none) -> HL0
- HL1: value (none) -> HL1
- HR0: value (none) -> HR0
- HR1: value (none) -> HR1
- PUMP0: value (none) -> PUMP0
- PUMP1: value (none) -> PUMP1
- REGULATOR: value (none) -> REGULATOR
- VL0: value (none) -> VL0
- VL1: value (none) -> VL1
- VR0: value (none) -> VR0
- VR1: value (none) -> VR1
- renumbered JP1 to REGULATOR
Connections:
- removed net N$3: PCB1.GPIO21
- removed net N$8: REGULATOR.EN
Changed lines of the file:
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@@
 <parts>
 <part name="PCB1" library="spencer" deviceset="RPI3" device=""/>
-<part name="JP1" library="spencer" deviceset="POLULU5VREGULATOR" device=""/>
+<part name="REGULATOR" library="spencer" deviceset="POLULU5VREGULATOR" device="" value="REGULATOR"/>
 <part name="ADC0" library="spencer" deviceset="MCP3208" device=""/>
 <part name="ADC1" library="spencer" deviceset="MCP3208" device=""/>
@@
 <part name="MOSFET1" library="SparkFun-DiscreteSemi" deviceset="MOSFET-NCHANNEL" device="FQP30N06L"/>
 <part name="MOSFET0" library="SparkFun-DiscreteSemi" deviceset="MOSFET-NCHANNEL" device="FQP30N06L"/>
-<part name="PUMP1" library="pinhead" deviceset="PINHD-1X2" device=""/>
-<part name="PUMP0" library="pinhead" deviceset="PINHD-1X2" device=""/>
+<part name="PUMP1" library="pinhead" deviceset="PINHD-1X2" device="" value="PUMP1"/>
+<part name="PUMP0" library="pinhead" deviceset="PINHD-1X2" device="" value="PUMP0"/>
 <part name="D1" library="SparkFun-DiscreteSemi" deviceset="DIODE" device="1N4148" value="1N4148"/>
 <part name="D2" library="SparkFun-DiscreteSemi" deviceset="DIODE" device="1N4148" value="1N4148"/>
-<part name="HL1" library="pinhead" deviceset="PINHD-1X6" device=""/>
-<part name="VL1" library="pinhead" deviceset="PINHD-1X6" device=""/>
-<part name="VR1" library="pinhead" deviceset="PINHD-1X6" device=""/>
-<part name="HR1" library="pinhead" deviceset="PINHD-1X6" device=""/>
-<part name="HL0" library="pinhead" deviceset="PINHD-1X6" device=""/>
-<part name="VL0" library="pinhead" deviceset="PINHD-1X6" device=""/>
-<part name="VR0" library="pinhead" deviceset="PINHD-1X6" device=""/>
-<part name="HR0" library="pinhead" deviceset="PINHD-1X6" device=""/>
-<part name="GND" library="pinhead" deviceset="PINHD-1X8" device=""/>
-<part name="AIN" library="pinhead" deviceset="PINHD-1X8" device=""/>
-<part name="3V3" library="pinhead" deviceset="PINHD-1X8" device=""/>
+<part name="HL1" library="pinhead" deviceset="PINHD-1X6" device="" value="HL1"/>
+<part name="VL1" library="pinhead" deviceset="PINHD-1X6" device="" value="VL1"/>
+<part name="VR1" library="pinhead" deviceset="PINHD-1X6" device="" value="VR1"/>
+<part name="HR1" library="pinhead" deviceset="PINHD-1X6" device="" value="HR1"/>
+<part name="HL0" library="pinhead" deviceset="PINHD-1X6" device="" value="HL0"/>
+<part name="VL0" library="pinhead" deviceset="PINHD-1X6" device="" value="VL0"/>
+<part name="VR0" library="pinhead" deviceset="PINHD-1X6" device="" value="VR0"/>
+<part name="HR0" library="pinhead" deviceset="PINHD-1X6" device="" value="HR0"/>
+<part name="GND" library="pinhead" deviceset="PINHD-1X8" device="" value="GND"/>
+<part name="AIN" library="pinhead" deviceset="PINHD-1X8" device="" value="AIN"/>
+<part name="3V3" library="pinhead" deviceset="PINHD-1X8" device="" value="3v3"/>
 </parts>
 <sheets>
@@
 <instances>
 <instance part="PCB1" gate="G$1" x="0" y="0"/>
-<instance part="JP1" gate="A" x="27.94" y="71.12"/>
+<instance part="REGULATOR" gate="A" x="27.94" y="71.12"/>
 <instance part="ADC0" gate="MCP3208$1" x="-53.34" y="-58.42"/>
 <instance part="ADC1" gate="MCP3208$1" x="-2.54" y="-60.96"/>
@@
 <net name="5V" class="0">
 <segment>
-<pinref part="JP1" gate="A" pin="VOUT"/>
+<pinref part="REGULATOR" gate="A" pin="VOUT"/>
 <junction x="27.94" y="66.04"/>
 <label x="22.86" y="66.04" size="1.27" layer="95" rot="MR0" xref="yes"/>
@@
 <net name="GND" class="0">
 <segment>
-<pinref part="JP1" gate="A" pin="GND2"/>
+<pinref part="REGULATOR" gate="A" pin="GND2"/>
 <junction x="27.94" y="68.58"/>
 <label x="22.86" y="68.58" size="1.27" layer="95" rot="MR0" xref="yes"/>
@@
 </segment>
 <segment>
-<pinref part="JP1" gate="A" pin="GND1"/>
+<pinref part="REGULATOR" gate="A" pin="GND1"/>
 <junction x="27.94" y="71.12"/>
 <label x="22.86" y="71.12" size="1.27" layer="95" rot="MR0" xref="yes"/>
@@
 </segment>
 </net>
-<net name="N$8" class="0">
-<segment>
-<pinref part="JP1" gate="A" pin="EN"/>
-<junction x="27.94" y="76.2"/>
-</segment>
-</net>
 <net name="PUMP1" class="0">
 <segment>
@@
 <pinref part="J1" gate="G$1" pin="PWR"/>
 <junction x="5.08" y="73.66"/>
-<pinref part="JP1" gate="A" pin="VIN"/>
+<pinref part="REGULATOR" gate="A" pin="VIN"/>
 <junction x="27.94" y="73.66"/>
 <wire x1="5.08" y1="73.66" x2="27.94" y2="73.66" width="0.1524" layer="91"/>
@@
 <junction x="-48.26" y="55.88"/>
 <label x="-53.34" y="55.88" size="1.27" layer="95" rot="R180" xref="yes"/>
+<wire x1="-48.26" y1="55.88" x2="-53.34" y2="55.88" width="0.1524" layer="91"/>
 </segment>
 <segment>
@@
 <junction x="-48.26" y="88.9"/>
 <label x="-53.34" y="88.9" size="1.27" layer="95" rot="R180" xref="yes"/>
+<wire x1="-48.26" y1="88.9" x2="-53.34" y2="88.9" width="0.1524" layer="91"/>
 </segment>
 <segment>
@@
 <wire x1="-20.32" y1="-152.4" x2="-2.54" y2="-152.4" width="0.1524" layer="91"/>
 <wire x1="-2.54" y1="-152.4" x2="-2.54" y2="-71.12" width="0.1524" layer="91"/>
-</segment>
-</net>
-<net name="N$3" class="0">
-<segment>
-<pinref part="PCB1" gate="G$1" pin="GPIO21"/>
-<junction x="48.26" y="15.24"/>
-<label x="48.26" y="17.78" size="1.27" layer="95" rot="R90" xref="yes"/>
 </segment>
 </net>
@@
 </sheet>
 </sheets>
+<errors>
+</errors>
 </schematic>
 </drawing>
