File: lever-arena.sch (EAGLE design)
At the start: 29 parts, among them J1 POWER_JACKPTH_BREAD

Commit message: REVISION 2.5
Parts:
- removed JP1, JP2, JP3, JP4: (no value), pinhead:PINHD-1X5
- added LL0: LL0, pinhead:PINHD-1X5
- added LL1: LL1, pinhead:PINHD-1X5
- added RL0: RL0, pinhead:PINHD-1X5
- added RL1: RL1, pinhead:PINHD-1X5
- added U$1, U$2, U$3, U$4: SPDTSWITCH, spencer:SPDTSWITCH
Connections:
- new net N$10: BNC2.1, U$3.P
- new net N$11: BNC3.1, U$4.P
- new net N$6: BNC0.1, U$1.P
- new net N$9: BNC1.1, U$2.P
- net 3V3: now also LL0.1, LL1.1, RL0.1, RL1.1; no longer JP1.1, JP2.1, JP3.1, JP4.1
- net 5V: now also LL0.5, LL1.5, RL0.5, RL1.5; no longer JP1.5, JP2.5, JP3.5, JP4.5
- net GND: now also LL0.4, LL1.4, RL0.4, RL1.4; no longer JP1.4, JP2.4, JP3.4, JP4.4
- net N$1: now also U$3.O
- net N$13: now also LL0.3; no longer JP1.3
- net N$14: now also LL0.2; no longer JP1.2
- net N$15: now also RL0.3; no longer JP2.3
- net N$17: now also RL0.2; no longer JP2.2
- net N$33: now also LL1.3, U$2.S; no longer JP3.3
- net N$34: now also LL1.2, U$1.S; no longer JP3.2
- net N$39: now also RL1.3, U$4.S; no longer JP4.3
- net N$40: now also RL1.2, U$3.S; no longer JP4.2
- net N$5: now also U$4.O
- net N$7: now also U$2.O
- net N$8: now also U$1.O
Other:
- moved on the sheet: BNC0, BNC1, BNC2, BNC3

Commit message: REVISION 2.6
To be sent for fabrication
Parts:
- added AUX: AUX, pinhead:PINHD-2X2
Connections:
- new net N$18: AUX.3, PCB1.GPIO23
- new net N$19: AUX.1, PCB1.GPIO24
- new net N$21: AUX.4, PCB1.GPIO25
- new net N$22: AUX.2, PCB1.GPIO21
Changed lines of the file:
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@@
 <part name="U$3" library="spencer" deviceset="SPDTSWITCH" device=""/>
 <part name="U$4" library="spencer" deviceset="SPDTSWITCH" device=""/>
+<part name="AUX" library="pinhead" deviceset="PINHD-2X2" device="" value="AUX"/>
 </parts>
 <sheets>
@@
 <instance part="U$3" gate="G$1" x="-71.12" y="-63.5" rot="R270"/>
 <instance part="U$4" gate="G$1" x="-71.12" y="-78.74" rot="R270"/>
+<instance part="AUX" gate="A" x="17.78" y="38.1"/>
 </instances>
 <busses>
@@
 </segment>
 </net>
+<net name="N$18" class="0">
+<segment>
+<pinref part="PCB1" gate="G$1" pin="GPIO23"/>
+<pinref part="AUX" gate="A" pin="3"/>
+<wire x1="-12.7" y1="38.1" x2="-12.7" y2="15.24" width="0.1524" layer="91"/>
+<wire x1="12.7" y1="38.1" x2="-12.7" y2="38.1" width="0.1524" layer="91"/>
+</segment>
+</net>
+<net name="N$19" class="0">
+<segment>
+<pinref part="PCB1" gate="G$1" pin="GPIO24"/>
+<wire x1="-7.62" y1="38.1" x2="-7.62" y2="35.56" width="0.1524" layer="91"/>
+<pinref part="AUX" gate="A" pin="1"/>
+<wire x1="-7.62" y1="35.56" x2="-7.62" y2="15.24" width="0.1524" layer="91"/>
+<wire x1="12.7" y1="40.64" x2="-7.62" y2="40.64" width="0.1524" layer="91"/>
+<wire x1="-7.62" y1="40.64" x2="-7.62" y2="38.1" width="0.1524" layer="91"/>
+</segment>
+</net>
+<net name="N$21" class="0">
+<segment>
+<pinref part="PCB1" gate="G$1" pin="GPIO25"/>
+<wire x1="2.54" y1="15.24" x2="2.54" y2="30.48" width="0.1524" layer="91"/>
+<wire x1="2.54" y1="30.48" x2="25.4" y2="30.48" width="0.1524" layer="91"/>
+<wire x1="25.4" y1="30.48" x2="25.4" y2="38.1" width="0.1524" layer="91"/>
+<pinref part="AUX" gate="A" pin="4"/>
+<wire x1="25.4" y1="38.1" x2="20.32" y2="38.1" width="0.1524" layer="91"/>
+</segment>
+</net>
+<net name="N$22" class="0">
+<segment>
+<pinref part="PCB1" gate="G$1" pin="GPIO21"/>
+<wire x1="48.26" y1="15.24" x2="48.26" y2="40.64" width="0.1524" layer="91"/>
+<pinref part="AUX" gate="A" pin="2"/>
+<wire x1="48.26" y1="40.64" x2="20.32" y2="40.64" width="0.1524" layer="91"/>
+</segment>
+</net>

Commit message: REVISION 2.7
Parts:
- added VSEL: VSEL, pinhead:PINHD-1X3
Connections:
- new net VA: HL0.3, HL1.3, HR0.3, HR1.3, VL0.3, VL1.3, VR0.3, VR1.3, VSEL.2
- net 12V: now also VSEL.1
- net 3V3: no longer PCB1.3V3@1
- net 5V: now also VSEL.3; no longer HL0.3, HL1.3, HR0.3, HR1.3, VL0.3, VL1.3, VR0.3, VR1.3
Changed lines of the file:
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@@
 <part name="U$4" library="spencer" deviceset="SPDTSWITCH" device=""/>
 <part name="AUX" library="pinhead" deviceset="PINHD-2X2" device="" value="AUX"/>
+<part name="VSEL" library="pinhead" deviceset="PINHD-1X3" device="" value="VSEL"/>
 </parts>
 <sheets>
@@
 <instance part="U$4" gate="G$1" x="-71.12" y="-78.74" rot="R270"/>
 <instance part="AUX" gate="A" x="17.78" y="38.1"/>
+<instance part="VSEL" gate="A" x="88.9" y="-78.74"/>
 </instances>
 <busses>
@@
 </segment>
 <segment>
-<pinref part="HR1" gate="A" pin="3"/>
-<junction x="121.92" y="-81.28"/>
-<label x="116.84" y="-81.28" size="1.778" layer="95" rot="R180"/>
-</segment>
-<segment>
-<pinref part="VR1" gate="A" pin="3"/>
-<junction x="121.92" y="-104.14"/>
-<label x="116.84" y="-104.14" size="1.778" layer="95" rot="R180"/>
-</segment>
-<segment>
-<pinref part="VL1" gate="A" pin="3"/>
-<junction x="121.92" y="-127"/>
-<label x="116.84" y="-127" size="1.778" layer="95" rot="R180"/>
-</segment>
-<segment>
-<pinref part="HL1" gate="A" pin="3"/>
-<junction x="121.92" y="-149.86"/>
-<label x="116.84" y="-149.86" size="1.778" layer="95" rot="R180"/>
-</segment>
-<segment>
-<pinref part="HR0" gate="A" pin="3"/>
-<junction x="154.94" y="-147.32"/>
-<label x="160.02" y="-147.32" size="1.778" layer="95"/>
-</segment>
-<segment>
-<pinref part="VR0" gate="A" pin="3"/>
-<junction x="154.94" y="-124.46"/>
-<label x="160.02" y="-124.46" size="1.778" layer="95"/>
-</segment>
-<segment>
-<pinref part="VL0" gate="A" pin="3"/>
-<junction x="154.94" y="-101.6"/>
-<label x="160.02" y="-101.6" size="1.778" layer="95"/>
-</segment>
-<segment>
-<pinref part="HL0" gate="A" pin="3"/>
-<junction x="154.94" y="-78.74"/>
-<label x="160.02" y="-78.74" size="1.778" layer="95"/>
-</segment>
-<segment>
 <pinref part="LL0" gate="A" pin="5"/>
 <junction x="30.48" y="-43.18"/>
@@
 <junction x="-12.7" y="-73.66"/>
 <label x="-17.78" y="-73.66" size="1.778" layer="95" rot="MR0"/>
+</segment>
+<segment>
+<pinref part="VSEL" gate="A" pin="3"/>
+<junction x="86.36" y="-81.28"/>
+<label x="76.2" y="-81.28" size="1.778" layer="95"/>
 </segment>
 </net>
@@
 <junction x="-7.62" y="-12.7"/>
 <label x="-7.62" y="-15.24" size="1.27" layer="95" rot="R270" xref="yes"/>
-</segment>
-<segment>
-<pinref part="PCB1" gate="G$1" pin="3V3@1"/>
-<junction x="-48.26" y="-12.7"/>
-<label x="-48.26" y="-15.24" size="1.27" layer="95" rot="R270" xref="yes"/>
 </segment>
 <segment>
@@
 <junction x="-63.5" y="50.8"/>
 <label x="-60.96" y="50.8" size="1.27" layer="95" xref="yes"/>
+</segment>
+<segment>
+<pinref part="VSEL" gate="A" pin="1"/>
+<junction x="86.36" y="-76.2"/>
+<label x="76.2" y="-76.2" size="1.778" layer="95"/>
 </segment>
 </net>
@@
 </segment>
 </net>
+<net name="VA" class="0">
+<segment>
+<pinref part="VSEL" gate="A" pin="2"/>
+<junction x="86.36" y="-78.74"/>
+<label x="76.2" y="-78.74" size="1.778" layer="95"/>
+</segment>
+<segment>
+<pinref part="HR1" gate="A" pin="3"/>
+<junction x="121.92" y="-81.28"/>
+<label x="116.84" y="-81.28" size="1.778" layer="95" rot="R180"/>
+</segment>
+<segment>
+<pinref part="VR1" gate="A" pin="3"/>
+<junction x="121.92" y="-104.14"/>
+<label x="116.84" y="-104.14" size="1.778" layer="95" rot="R180"/>
+</segment>
+<segment>
+<pinref part="VL1" gate="A" pin="3"/>
+<junction x="121.92" y="-127"/>
+<label x="116.84" y="-127" size="1.778" layer="95" rot="R180"/>
+</segment>
+<segment>
+<pinref part="HL1" gate="A" pin="3"/>
+<junction x="121.92" y="-149.86"/>
+<label x="116.84" y="-149.86" size="1.778" layer="95" rot="R180"/>
+</segment>
+<segment>
+<pinref part="HR0" gate="A" pin="3"/>
+<junction x="154.94" y="-147.32"/>
+<label x="160.02" y="-147.32" size="1.778" layer="95"/>
+</segment>
+<segment>
+<pinref part="VR0" gate="A" pin="3"/>
+<junction x="154.94" y="-124.46"/>
+<label x="160.02" y="-124.46" size="1.778" layer="95"/>
+</segment>
+<segment>
+<pinref part="VL0" gate="A" pin="3"/>
+<junction x="154.94" y="-101.6"/>
+<label x="160.02" y="-101.6" size="1.778" layer="95"/>
+</segment>
+<segment>
+<pinref part="HL0" gate="A" pin="3"/>
+<junction x="154.94" y="-78.74"/>
+<label x="160.02" y="-78.74" size="1.778" layer="95"/>
+</segment>
+</net>
