File: lever-arena.brd (EAGLE design)
At the start: 77 x 56 mm, 33 parts, among them J1 POWER_JACKPTH_BREAD

Commit message: REVISION 2.6
To be sent for fabrication
Parts:
- added AUX: AUX, pinhead:2X02
Connections:
- new net N$18: AUX.3, PCB1.P$16
- new net N$19: AUX.1, PCB1.P$18
- new net N$21: AUX.4, PCB1.P$22
- new net N$22: AUX.2, PCB1.P$40
Routing:
- net N$18: track 0.00 -> 84.0 mm
- net N$19: track 0.00 -> 81.2 mm
- net N$21: track 0.00 -> 70.2 mm
- net N$22: track 0.00 -> 45.5 mm
- net N$39: track 107.6 -> 109.2 mm
- net N$40: track 120.7 -> 122.1 mm
- net 5V: track 213.4 -> 212.3 mm
Other:
- board text added: "Lever-Arena io board Revision 2.6 Spencer Boyer boyer2@uw.edu"
- board text removed: "Lever-Arena io board Revision 2.5 Spencer Boyer boyer2@uw.edu"
Changed lines of the file:
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@@
 <text x="61.4" y="13.3" size="1" layer="25" rot="R270">AIN</text>
 <text x="75.8" y="6.4" size="1" layer="25" font="vector" rot="R180">Lever-Arena io board
-Revision 2.5
+Revision 2.6
 Spencer Boyer
 boyer2@uw.edu</text>
@@
 <element name="U$3" library="spencer" package="JS202011CQNSPDT" value="SPDTSWITCH" x="13.8" y="25" rot="R270"/>
 <element name="U$4" library="spencer" package="JS202011CQNSPDT" value="SPDTSWITCH" x="10.5" y="12.3"/>
+<element name="AUX" library="pinhead" package="2X02" value="AUX" x="73.5" y="9.6"/>
 </elements>
 <signals>
@@
 <wire x1="39.955" y1="49.739790625" x2="39.88060625" y2="49.91939375" width="0.254" layer="1" curve="44.999502"/>
 <wire x1="39.88060625" y1="49.91939375" x2="39.5" y2="50.3" width="0.254" layer="1"/>
-<wire x1="39.5" y1="50.3" x2="39.5" y2="54.594790625" width="0.254" layer="1"/>
-<wire x1="39.5" y1="54.594790625" x2="39.42560625" y2="54.77439375" width="0.254" layer="1" curve="44.999502"/>
-<wire x1="39.42560625" y1="54.77439375" x2="38.6" y2="55.6" width="0.254" layer="1"/>
-<wire x1="38.6" y1="55.6" x2="22.290009375" y2="55.6" width="0.254" layer="1"/>
-<wire x1="22.290009375" y1="55.6" x2="22.11040625" y2="55.52560625" width="0.254" layer="1" curve="44.999502"/>
-<wire x1="22.11040625" y1="55.52560625" x2="20.3566" y2="53.7718" width="0.254" layer="1"/>
 <wire x1="20.3566" y1="53.7718" x2="18.4718" y2="53.7718" width="1.5" layer="16"/>
 <wire x1="18.4718" y1="53.7718" x2="18" y2="53.3" width="1.5" layer="16"/>
@@
 <wire x1="40" y1="47.755" x2="39.955" y2="47.8" width="0.254" layer="1"/>
 <wire x1="22.8966" y1="53.7718" x2="20.3566" y2="53.7718" width="1.5" layer="16"/>
+<wire x1="39.5" y1="50.3" x2="39.5" y2="52.1" width="0.254" layer="1"/>
+<wire x1="39.5" y1="52.1" x2="39.2" y2="52.4" width="0.254" layer="1"/>
+<wire x1="39.2" y1="52.4" x2="30" y2="52.4" width="0.254" layer="1"/>
+<wire x1="30" y1="52.4" x2="29.3" y2="53.1" width="0.254" layer="1"/>
+<wire x1="29.3" y1="53.1" x2="29.3" y2="54.4" width="0.254" layer="1"/>
+<wire x1="29.3" y1="54.4" x2="28.6" y2="55.1" width="0.254" layer="1"/>
+<wire x1="28.6" y1="55.1" x2="21.6848" y2="55.1" width="0.254" layer="1"/>
+<wire x1="21.6848" y1="55.1" x2="20.3566" y2="53.7718" width="0.254" layer="1"/>
 </signal>
 <signal name="GND">
@@
 <contactref element="U$4" pad="P$4"/>
 <contactref element="U$4" pad="P$2"/>
-<wire x1="13" y1="10.65" x2="13" y2="2.6" width="0.254" layer="1"/>
-<wire x1="13" y1="2.6" x2="15" y2="0.6" width="0.254" layer="1"/>
-<wire x1="15" y1="0.6" x2="48.8" y2="0.6" width="0.254" layer="1"/>
+<wire x1="11.8" y1="2.7" x2="13.8" y2="0.7" width="0.254" layer="1"/>
+<wire x1="13.8" y1="0.7" x2="48.8" y2="0.6" width="0.254" layer="1"/>
 <wire x1="48.8" y1="0.6" x2="50.6" y2="2.4" width="0.254" layer="1"/>
 <wire x1="50.6" y1="2.4" x2="50.6" y2="16.2" width="0.254" layer="1"/>
 <wire x1="50.6" y1="16.2" x2="50.8" y2="16.4" width="0.254" layer="1"/>
 <wire x1="13" y1="13.95" x2="13" y2="10.65" width="0.254" layer="1"/>
+<wire x1="11.8" y1="2.7" x2="11.8" y2="9.45" width="0.254" layer="1"/>
+<wire x1="11.8" y1="9.45" x2="13" y2="10.65" width="0.254" layer="1"/>
 </signal>
 <signal name="N$40">
@@
 <wire x1="12.15" y1="22.5" x2="12.15" y2="16.35" width="0.254" layer="16"/>
 <wire x1="12.15" y1="16.35" x2="14.7" y2="13.8" width="0.254" layer="16"/>
-<wire x1="14.2" y1="6.8" x2="13.5" y2="6.1" width="0.254" layer="1"/>
-<wire x1="13.5" y1="6.1" x2="13.5" y2="2.9" width="0.254" layer="1"/>
-<wire x1="13.5" y1="2.9" x2="15.3" y2="1.2" width="0.254" layer="1"/>
-<wire x1="15.3" y1="1.2" x2="48.3" y2="1.2" width="0.254" layer="1"/>
+<wire x1="13.8" y1="7.6" x2="12.5" y2="6.1" width="0.254" layer="1"/>
+<wire x1="12.5" y1="6.1" x2="12.5" y2="2.9" width="0.254" layer="1"/>
+<wire x1="12.5" y1="2.9" x2="14.1" y2="1.3" width="0.254" layer="1"/>
+<wire x1="14.1" y1="1.3" x2="48.3" y2="1.2" width="0.254" layer="1"/>
 <wire x1="48.3" y1="1.2" x2="50" y2="2.8" width="0.254" layer="1"/>
 <wire x1="50" y1="2.8" x2="50" y2="15.76" width="0.254" layer="1"/>
 <wire x1="50" y1="15.76" x2="46.56" y2="19.2" width="0.254" layer="1"/>
-<via x="14.2" y="6.8" extent="1-16" drill="0.4"/>
-<wire x1="14.7" y1="13.8" x2="14.7" y2="7.3" width="0.254" layer="16"/>
-<wire x1="14.7" y1="7.3" x2="14.2" y2="6.8" width="0.254" layer="16"/>
+<via x="13.8" y="7.6" extent="1-16" drill="0.4"/>
+<wire x1="14.7" y1="13.8" x2="14.7" y2="8.6" width="0.254" layer="16"/>
+<wire x1="14.7" y1="8.6" x2="13.8" y2="7.6" width="0.254" layer="16"/>
 <wire x1="12.15" y1="22.5" x2="15.45" y2="22.5" width="0.254" layer="1"/>
 </signal>
@@
 <wire x1="10.5" y1="13.95" x2="10.5" y2="10.65" width="0.254" layer="1"/>
 </signal>
+<signal name="N$18">
+<contactref element="PCB1" pad="P$16"/>
+<wire x1="38.1366" y1="53.7718" x2="38.1366" y2="54.0366" width="0.254" layer="1"/>
+<wire x1="38.1366" y1="54.0366" x2="39.4" y2="55.3" width="0.254" layer="1"/>
+<wire x1="39.4" y1="55.3" x2="68.7" y2="55.3" width="0.254" layer="1"/>
+<wire x1="68.7" y1="55.3" x2="70.1" y2="53.9" width="0.254" layer="1"/>
+<wire x1="70.1" y1="53.9" x2="70.1" y2="50.6" width="0.254" layer="1"/>
+<wire x1="70.1" y1="50.6" x2="70.5" y2="50.2" width="0.254" layer="1"/>
+<wire x1="70.5" y1="50.2" x2="72.4" y2="50.2" width="0.254" layer="1"/>
+<wire x1="72.4" y1="50.2" x2="76" y2="46.6" width="0.254" layer="1"/>
+<wire x1="76" y1="46.6" x2="76" y2="14.5" width="0.254" layer="1"/>
+<wire x1="76" y1="14.5" x2="73.5" y2="12" width="0.254" layer="1"/>
+<wire x1="73.5" y1="12" x2="73.5" y2="9.6" width="0.254" layer="1"/>
+<contactref element="AUX" pad="3"/>
+<wire x1="73.5" y1="9.6" x2="74.77" y2="8.33" width="0.254" layer="1"/>
+</signal>
+<signal name="N$19">
+<contactref element="PCB1" pad="P$18"/>
+<wire x1="40.6766" y1="53.7718" x2="40.6766" y2="53.7766" width="0.254" layer="1"/>
+<wire x1="40.6766" y1="53.7766" x2="41.7" y2="54.8" width="0.254" layer="1"/>
+<wire x1="41.7" y1="54.8" x2="66.9" y2="54.8" width="0.254" layer="1"/>
+<wire x1="66.9" y1="54.8" x2="67.3" y2="54.4" width="0.254" layer="1"/>
+<wire x1="67.3" y1="54.4" x2="67.3" y2="50.9" width="0.254" layer="1"/>
+<wire x1="67.3" y1="50.9" x2="68.6" y2="49.6" width="0.254" layer="1"/>
+<wire x1="68.6" y1="49.6" x2="72" y2="49.6" width="0.254" layer="1"/>
+<wire x1="72" y1="49.6" x2="75.4" y2="46.2" width="0.254" layer="1"/>
+<wire x1="75.4" y1="46.2" x2="75.4" y2="17.6" width="0.254" layer="1"/>
+<wire x1="75.4" y1="17.6" x2="70.8" y2="13" width="0.254" layer="1"/>
+<contactref element="AUX" pad="1"/>
+<wire x1="70.8" y1="13" x2="70.8" y2="9.66" width="0.254" layer="1"/>
+<wire x1="70.8" y1="9.66" x2="72.23" y2="8.33" width="0.254" layer="1"/>
+</signal>
+<signal name="N$21">
+<contactref element="PCB1" pad="P$22"/>
+<contactref element="AUX" pad="4"/>
+<wire x1="74.77" y1="10.87" x2="74.77" y2="11.63" width="0.254" layer="16"/>
+<wire x1="74.77" y1="11.63" x2="72.8" y2="13.6" width="0.254" layer="16"/>
+<wire x1="72.8" y1="13.6" x2="72.8" y2="46.1" width="0.254" layer="16"/>
+<wire x1="72.8" y1="46.1" x2="70.1" y2="48.8" width="0.254" layer="16"/>
+<wire x1="70.1" y1="48.8" x2="70.1" y2="53.9" width="0.254" layer="16"/>
+<wire x1="70.1" y1="53.9" x2="69.1" y2="54.9" width="0.254" layer="16"/>
+<wire x1="69.1" y1="54.9" x2="46.8848" y2="54.9" width="0.254" layer="16"/>
+<wire x1="46.8848" y1="54.9" x2="45.7566" y2="53.7718" width="0.254" layer="16"/>
+</signal>
+<signal name="N$22">
+<contactref element="PCB1" pad="P$40"/>
+<contactref element="AUX" pad="2"/>
+<wire x1="72.23" y1="10.87" x2="72.23" y2="44.87" width="0.254" layer="16"/>
+<wire x1="72.23" y1="44.87" x2="67.3" y2="49.8" width="0.254" layer="16"/>
+<wire x1="67.3" y1="49.8" x2="67.3" y2="52.4552" width="0.254" layer="16"/>
+<wire x1="67.3" y1="52.4552" x2="68.6166" y2="53.7718" width="0.254" layer="16"/>
+</signal>
 </signals>

Commit message: REVISION 2.7
Parts:
- added VSEL: VSEL, pinhead:1X03
Connections:
- new net VA: HL0.3, HL1.3, HR0.3, HR1.3, VL0.3, VL1.3, VR0.3, VR1.3, VSEL.2
- net 12V: now also VSEL.1
- net 3V3: no longer PCB1.P$1
- net 5V: now also VSEL.3; no longer HL0.3, HL1.3, HR0.3, HR1.3, VL0.3, VL1.3, VR0.3, VR1.3
Routing:
- net 5V: track 212.3 -> 167.7 mm, vias 1 -> 2
- net VA: track 0.00 -> 41.1 mm
- net 12V: track 86.4 -> 112.9 mm
- net GND: track 401.6 -> 384.7 mm
- net N$40: track 122.1 -> 113.7 mm
- net N$39: track 109.2 -> 102.4 mm
- net N$33: track 122.8 -> 122.2 mm
Other:
- board text added: "12V"
- board text added: "Lever-Arena io board Revision 2.7 Spencer Boyer boyer2@uw.edu"
- board text added: "VA"
- board text removed: "Lever-Arena io board Revision 2.6 Spencer Boyer boyer2@uw.edu"
